File: Valve-PCB-Eagle/ValveDriver-8ch.brd (EAGLE design)
At the start: 101.6 x 76.2 mm, 27 parts, among them IC1 ULQ2803A, J10 Valve 3, J11 Valve 2, J12 Valve 1, J15 BNCPTH, J16 BNCPTH, J17 BNCPTH, J18 BNCPTH, J4 POWER_JACK, J5 Valve 8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

Commit message: [Valve] Removed Teensy and associated I/O connections
Parts:
- removed J3: (no value), SparkFun-Connectors:1X08
- removed JP1: JUMPER-SMT_2_NO_SILK, SparkFun-Jumpers:SMT-JUMPER_2_NO_SILK
- removed U$1: TEENSY_3.1-3.2_DIL, Teensy_3_and_LC_Series_Boards_v1.4:TEENSY_3.0-3.2&LC_DIL
- moved U$7 60.8 mm to (21.6, 16.5)
- moved J1 39.6 mm to (97.8, 12.7), turned to 90 degrees
- moved U$2 25.4 mm to (96.5, 45.7)
- moved U$6 25.4 mm to (5.08, 45.7)
- moved J15 25.4 mm to (85.1, 39.4)
- moved J16 25.4 mm to (62.2, 39.4)
- moved J17 25.4 mm to (39.4, 39.4)
- moved J18 25.4 mm to (16.5, 39.4)
- moved S1 22.9 mm to (15.2, 29.2)
- moved S2 22.9 mm to (39.4, 29.2)
- moved S3 22.9 mm to (63.5, 29.2)
- moved S4 22.9 mm to (86.4, 29.2)
- moved IC1 10.2 mm to (43.2, 16.5)
- moved J12 7.62 mm to (14.0, 5.08)
- moved J11 6.35 mm to (24.1, 5.08)
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Connections:
- removed net 3.3V: J3.7, U$1.3.3V
- removed net AGND: U$1.AGND
- removed net IO_1: J3.6, U$1.11
- removed net IO_2: J3.5, U$1.12
- removed net IO_3: J3.4, U$1.14/A0
- removed net IO_4: J3.3, U$1.15/A1
- removed net V_IN_TEENSY: J3.8, JP1.1, U$1.VIN
- net GND: no longer J3.1, J3.2, U$1.GND
- net V1: no longer U$1.3
- net V2: no longer U$1.4
- net V3: no longer U$1.5
- net V4: no longer U$1.6
- net V5: no longer U$1.9
- net V6: no longer U$1.10
- net V7: no longer U$1.20/A6
- net V8: no longer U$1.21/A7
- net V_VALVE: no longer JP1.2
Routing:
- net V_IN_TEENSY: track 74.0 -> 0.00 mm
- net V8: track 108.1 -> 50.0 mm
- net 3.3V: track 47.9 -> 0.00 mm
- net V3: track 114.9 -> 73.3 mm, vias 2 -> 0
- net V1OUT: track 88.5 -> 47.1 mm
- net V7: track 90.3 -> 51.2 mm
- net V2: track 114.9 -> 81.2 mm, vias 3 -> 0
- net V1: track 118.0 -> 92.0 mm, vias 1 -> 0
- net V3OUT: track 66.2 -> 41.0 mm
- net V4: track 101.7 -> 77.1 mm, vias 2 -> 0
- net V4OUT: track 83.3 -> 58.9 mm
- net V2OUT: track 65.6 -> 42.5 mm
- net IO_1: track 22.5 -> 0.00 mm, vias 1 -> 0
- net IO_4: track 22.4 -> 0.00 mm
- net IO_3: track 19.4 -> 0.00 mm
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Other:
- board size 101.6 x 76.2 mm -> 101.6 x 50.8 mm
- board text added: "Valve Activation Buttons"
- board text removed: "(External inputs or from Teensy)"
- board text removed: "Close jumper to power Teensy from V_valve. (If closed, do not connect Teensy to USB power.)"
- board text removed: "General purpose input/output lines for Teensy"
- board text removed: "Gnd Gnd IO_4 IO_3 IO_2 IO_1 3.3V Vin/5V"
- board text removed: "V1 V2 V3 V4 V5 V6 IO_1 IO_2"
- board text removed: "V1 V2 V3 V4 V5 V6 V7 V8"
- board text removed: "V8 V7 IO_4 IO_3"
- board text removed: "with optional Teensy control"
